File: MotorControlShield_MK2.kicad_sch (KiCad schematic)
At the start: 66 parts, among them J1 Screw_Terminal_01x02, J2 Screw_Terminal_01x02, J3 Screw_Terminal_01x02, J5 Screw_Terminal_01x02, Q1 IRLIZ44N, Q10 QM6006D, Q2 QM6006D, Q4 QM6006D, Q5 IRLIZ44N, Q6 IRLIZ44N, Q8 IRLIZ44N, Q9 QM6006D, U1 IR2110, U2 LM5109MA, U3 LM78M12_TO252, U5 LM5109MA, U6 IR2110, U7 BTN7960B, U8 BTN7960B

Commit message: Added documentation/layout
Other:
- note added: "BTN7960Bs are third option"
- note added: "Half bridge drivers: LM5109MA alternative"
- note added: "IR2110 are primary half bridge driver ICs"
- note added: "Single motor driver board half bridge options: IR2210 (primary) alternatives: BTN7960Bs or LM5109MAs For MOSFETs: TO-252s, TO-263s or TO-220s For the 12V : either direct 12V from external supply or on-board 12V regulator in TO-220 or TO-252 package 5V must be supplied externally"
Changed lines of the file:
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@@
+	)
+	(rectangle
+		(start 59.182 141.986)
+		(end 112.268 173.736)
+		(stroke
+			(width 0)
+			(type default)
+		)
+		(fill
+			(type none)
+		)
+	)
+	(rectangle
+		(start 199.39 88.646)
+		(end 252.476 120.396)
+		(stroke
+			(width 0)
+			(type default)
+		)
+		(fill
+			(type none)
+		)
+	)
+	(rectangle
+		(start 87.122 37.592)
+		(end 201.93 65.024)
+		(stroke
+			(width 0)
+			(type default)
+		)
+		(fill
+			(type none)
+		)
 	)
 	(rectangle
@@
 		(fill
 			(type none)
+		)
+	)
+	(text "BTN7960Bs are\nthird option"
+		(exclude_from_sim no)
+		(at 60.706 155.194 0)
+		(effects
+			(font
+				(size 1.27 1.27)
+			)
+			(justify left)
+		)
+	)
+	(text "Single motor driver board\nhalf bridge options: IR2210 (primary)\nalternatives: BTN7960Bs or LM5109MAs\n\nFor MOSFETs: TO-252s, TO-263s or TO-220s\n\nFor the 12V : either direct 12V from external supply or on-board\n12V regulator in TO-220 or TO-252 package\n\n5V must be supplied externally"
+		(exclude_from_sim no)
+		(at 277.622 130.048 0)
+		(effects
+			(font
+				(size 2.54 2.54)
+				(thickness 0.508)
+				(bold yes)
+			)
+			(justify left)
+		)
+	)
+	(text "Half bridge drivers: LM5109MA alternative"
+		(exclude_from_sim no)
+		(at 149.86 41.402 0)
+		(effects
+			(font
+				(size 1.27 1.27)
+			)
 		)
 	)
@@
 		(effects
 			(font
+				(size 1.27 1.27)
+			)
+			(justify left)
+		)
+	)
+	(text "IR2110 are primary half bridge\ndriver ICs"
+		(exclude_from_sim no)
+		(at 221.742 110.236 0)
+		(effects
+			(font

Commit message: Added pads for extra current
Parts:
- added C16, C18, C19, C21, C22, C23, C25, C27, C29, C30, C32, C33, C34, C36, C38, C40, C41, C43, C44, C45, C47: 100n, Capacitor_THT:C_Rect_L7.0mm_W3.5mm_P5.00mm, symbol Device:C
- added C17, C20, C24, C26, C28, C31, C35, C37, C39, C42, C46, C48: 10u, termocuplu:CP_Elec_6.3x3.9_COMPOSITE, symbol Device:C_Polarized
- added D10, D11, D12, D13, D14, D15, D16, D17, D18, D19, D20, D21, D22, D23, D24, D7, D8, D9: 1N4002, Diode_THT:D_DO-41_SOD81_P10.16mm_Horizontal, symbol Diode:1N4002
- added J10, J4, J6, J7, J8, J9: Screw_Terminal_01x02, TO220:TerminalBlock_CLEAN_2PIN, symbol Connector:Screw_Terminal_01x02
- added Q11, Q13, Q16, Q18, Q19, Q21, Q24, Q26, Q27, Q29, Q32, Q7: QM6006D, Package_TO_SOT_SMD:TO-263-2, symbol Transistor_FET:QM6006D
- added Q12, Q14, Q15, Q17, Q20, Q22, Q23, Q25, Q28, Q3, Q30, Q31: IRLIZ44N, TO220:TO-220-3_EXTENDED2, symbol Transistor_FET:IRLIZ44N
- added R17, R19, R31, R32, R33, R35, R47, R48, R49, R51, R63, R64: 10k, TO220:R_Axial_Clean, symbol Device:R
- added R18, R20, R21, R22, R23, R24, R25, R26, R27, R28, R29, R30, R34, R36, R37, R38, R39, R40, R41, R42, R43, R44, R45, R46, R50, R52, R53, R54, R55, R56, R57, R58, R59, R60, R61, R62: 1k, TO220:R_Axial_Clean, symbol Device:R
- added U10, U11, U16, U17, U22, U23: LM5109MA, Package_SO:SOIC-8_3.9x4.9mm_P1.27mm, symbol Driver_FET:LM5109MA
- added U12, U15, U18, U21, U24, U9: BTN7960B, termocuplu:IC_BTN7960B, symbol ktype:BTN7960B
- added U13, U14, U19, U20, U25, U4: IR2110, Package_DIP:DIP-14_W7.62mm, symbol Driver_FET:IR2110
Connections:
- net 12V: now also C19.1, C30.1, C41.1, D12.2 (A), D13.2 (A), D18.2 (A), D19.2 (A), D24.2 (A), D7.2 (A), U10.1 (VDD), U11.1 (VDD), U13.3 (VCC), U14.3 (VCC), U16.1 (VDD), U17.1 (VDD), U19.3 (VCC), U20.3 (VCC), U22.1 (VDD), U23.1 (VDD), U25.3 (VCC), U4.3 (VCC)
- net 5V: now also C16.1, C17.1, C25.1, C26.1, C27.1, C28.1, C36.1, C37.1, C38.1, C39.1, C47.1, C48.1, R17.2, R32.2, R33.2, R48.2, R49.2, R64.2, U13.9 (VDD), U14.9 (VDD), U19.9 (VDD), U20.9 (VDD), U25.9 (VDD), U4.9 (VDD)
- net GND: now also C16.2, C17.2, C19.2, C21.2, C22.2, C25.2, C26.2, C27.2, C28.2, C30.2, C32.2, C33.2, C36.2, C37.2, C38.2, C39.2, C41.2, C43.2, C44.2, C47.2, C48.2, Q12.3 (S), Q13.3 (S), Q14.3 (S), Q18.3 (S), Q20.3 (S), Q21.3 (S), Q22.3 (S), Q26.3 (S), Q28.3 (S), Q29.3 (S), Q30.3 (S), Q7.3 (S), R18.1, R22.1, R23.1, R26.1, R27.1, R30.1, R34.1, R38.1, R39.1, R42.1, R43.1, R46.1, R50.1, R54.1, R55.1, R58.1, R59.1, R62.1, U10.4 (VSS), U11.4 (VSS), U12.1 (GND), U13.11 (SD), U13.13 (VSS), U13.2 (COM), U14.11 (SD), U14.13 (VSS), U14.2 (COM), U15.1 (GND), U16.4 (VSS), U17.4 (VSS), U18.1 (GND), U19.11 (SD), U19.13 (VSS), U19.2 (COM), U20.11 (SD), U20.13 (VSS), U20.2 (COM), U21.1 (GND), U22.4 (VSS), U23.4 (VSS), U24.1 (GND), U25.11 (SD), U25.13 (VSS), U25.2 (COM), U4.11 (SD), U4.13 (VSS), U4.2 (COM), U9.1 (GND)
- net VDC: now also C21.1, C22.1, C32.1, C33.1, C43.1, C44.1, Q11.2 (D), Q15.2 (D), Q16.2 (D), Q17.2 (D), Q19.2 (D), Q23.2 (D), Q24.2 (D), Q25.2 (D), Q27.2 (D), Q3.2 (D), Q31.2 (D), Q32.2 (D), U12.7 (VS), U15.7 (VS), U18.7 (VS), U21.7 (VS), U24.7 (VS), U9.7 (VS)
- new net: D21.2 (A), Q25.1 (G), Q27.1 (G), R52.1, R56.2
- new net: D21.1 (K), R52.2, U20.7 (HO), U22.7 (HO)
- new net: D9.2 (A), Q11.1 (G), Q3.1 (G), R20.1, R24.2
- new net: D9.1 (K), R20.2, U10.7 (HO), U4.7 (HO)
- new net: D11.2 (A), Q13.1 (G), Q14.1 (G), R26.2, R29.1
- new net: C23.2, C24.2, J7.2 (Pin_2), Q13.2 (D), Q14.2 (D), Q15.3 (S), Q16.3 (S), R28.1, U11.6 (HS), U12.4 (OUT), U12.8 (OUT), U13.5 (VS)
- new net: J9.1 (Pin_1), R63.2, U20.10 (HIN), U22.2 (HI), U23.3 (LI), U25.12 (LIN)
- new net: J9.2 (Pin_2), R51.2, U20.12 (LIN), U22.3 (LI), U23.2 (HI), U25.10 (HIN)
- new net: D20.1 (K), R53.2, U20.1 (LO), U22.5 (LO)
- new net: C40.2, C42.2, J10.1 (Pin_1), Q25.3 (S), Q26.2 (D), Q27.3 (S), Q28.2 (D), R56.1, U20.5 (VS), U21.4 (OUT), U21.8 (OUT), U22.6 (HS)
- new net: C40.1, C42.1, D19.1 (K), U20.6 (VB), U22.8 (HB)
- new net: R34.2, U15.5 (SR)
- new net: R63.1, U24.2 (IN)
- new net: J4.2 (Pin_2), R19.2, U10.3 (LI), U11.2 (HI), U13.10 (HIN), U4.12 (LIN)
- new net: J4.1 (Pin_1), R31.2, U10.2 (HI), U11.3 (LI), U13.12 (LIN), U4.10 (HIN)
- new net: D11.1 (K), R29.2, U11.5 (LO), U13.1 (LO)
- new net: D10.1 (K), R25.2, U11.7 (HO), U13.7 (HO)
- new net: C23.1, C24.1, D12.1 (K), U11.8 (HB), U13.6 (VB)
- new net: R46.2, U18.5 (SR)
- new net: C34.2, C35.2, J8.2 (Pin_2), Q21.2 (D), Q22.2 (D), Q23.3 (S), Q24.3 (S), R44.1, U17.6 (HS), U18.4 (OUT), U18.8 (OUT), U19.5 (VS)
- new net: D16.2 (A), Q23.1 (G), Q24.1 (G), R41.1, R44.2
- new net: R64.1, U24.3 (INH)
- new net: C45.2, C46.2, J10.2 (Pin_2), Q29.2 (D), Q30.2 (D), Q31.3 (S), Q32.3 (S), R60.1, U23.6 (HS), U24.4 (OUT), U24.8 (OUT), U25.5 (VS)
- new net: R62.2, U24.5 (SR)
- new net: R59.2, U24.6 (IS)
- new net: D10.2 (A), Q15.1 (G), Q16.1 (G), R25.1, R28.2
- new net: R51.1, U21.2 (IN)
- new net: R49.1, U21.3 (INH)
- new net: R50.2, U21.5 (SR)
- new net: R54.2, U21.6 (IS)
- new net: D17.2 (A), Q21.1 (G), Q22.1 (G), R42.2, R45.1
- new net: D17.1 (K), R45.2, U17.5 (LO), U19.1 (LO)
- new net: D16.1 (K), R41.2, U17.7 (HO), U19.7 (HO)
- new net: D23.1 (K), R61.2, U23.5 (LO), U25.1 (LO)
- new net: D23.2 (A), Q29.1 (G), Q30.1 (G), R58.2, R61.1
- new net: D8.2 (A), Q12.1 (G), Q7.1 (G), R21.1, R23.2
- new net: D8.1 (K), R21.2, U10.5 (LO), U4.1 (LO)
- new net: D22.2 (A), Q31.1 (G), Q32.1 (G), R57.1, R60.2
- new net: J6.2 (Pin_2), R35.2, U14.12 (LIN), U16.3 (LI), U17.2 (HI), U19.10 (HIN)
- new net: J6.1 (Pin_1), R47.2, U14.10 (HIN), U16.2 (HI), U17.3 (LI), U19.12 (LIN)
- new net: C34.1, C35.1, D18.1 (K), U17.8 (HB), U19.6 (VB)
- new net: C29.1, C31.1, D13.1 (K), U14.6 (VB), U16.8 (HB)
- new net: C29.2, C31.2, J8.1 (Pin_1), Q17.3 (S), Q18.2 (D), Q19.3 (S), Q20.2 (D), R40.1, U14.5 (VS), U15.4 (OUT), U15.8 (OUT), U16.6 (HS)
- new net: D20.2 (A), Q26.1 (G), Q28.1 (G), R53.1, R55.2
- new net: D22.1 (K), R57.2, U23.7 (HO), U25.7 (HO)
- new net: R22.2, U9.6 (IS)
- new net: D14.2 (A), Q18.1 (G), Q20.1 (G), R37.1, R39.2
- new net: D14.1 (K), R37.2, U14.1 (LO), U16.5 (LO)
- new net: R33.1, U15.3 (INH)
- new net: C45.1, C46.1, D24.1 (K), U23.8 (HB), U25.6 (VB)
- new net: R43.2, U18.6 (IS)
- new net: R38.2, U15.6 (IS)
- new net: R32.1, U12.3 (INH)
- new net: R18.2, U9.5 (SR)
- new net: C18.2, C20.2, J7.1 (Pin_1), Q11.3 (S), Q12.2 (D), Q3.3 (S), Q7.2 (D), R24.1, U10.6 (HS), U4.5 (VS), U9.4 (OUT), U9.8 (OUT)
- new net: C18.1, C20.1, D7.1 (K), U10.8 (HB), U4.6 (VB)
- new net: R35.1, U15.2 (IN)
- new net: D15.2 (A), Q17.1 (G), Q19.1 (G), R36.1, R40.2
- new net: D15.1 (K), R36.2, U14.7 (HO), U16.7 (HO)
- new net: R17.1, U9.3 (INH)
- new net: R19.1, U9.2 (IN)
- new net: R47.1, U18.2 (IN)
- new net: R48.1, U18.3 (INH)
- new net: R27.2, U12.6 (IS)
- new net: R30.2, U12.5 (SR)
- new net: R31.1, U12.2 (IN)
Other:
- note added: "Motor 1"
- note added: "Motor 2"
- note added: "Motor 3"
- note added: "Motor 4"

Commit message: Made self contained footprints
Parts:
- removed C16, C18, C19, C21, C22, C23, C25, C27, C29, C30, C32, C33, C34, C36, C38, C40, C41, C43, C44, C45, C47: 100n, Capacitor_THT:C_Rect_L7.0mm_W3.5mm_P5.00mm, symbol Device:C
- removed C17, C20, C24, C26, C28, C31, C35, C37, C39, C42, C46, C48: 10u, termocuplu:CP_Elec_6.3x3.9_COMPOSITE, symbol Device:C_Polarized
- removed D10, D11, D12, D13, D14, D15, D16, D17, D18, D19, D20, D21, D22, D23, D24, D7, D8, D9: 1N4002, Diode_THT:D_DO-41_SOD81_P10.16mm_Horizontal, symbol Diode:1N4002
- removed J10, J4, J6, J7, J8, J9: Screw_Terminal_01x02, TO220:TerminalBlock_CLEAN_2PIN, symbol Connector:Screw_Terminal_01x02
- removed Q11, Q13, Q16, Q18, Q19, Q21, Q24, Q26, Q27, Q29, Q32, Q7: QM6006D, Package_TO_SOT_SMD:TO-263-2, symbol Transistor_FET:QM6006D
- removed Q12, Q14, Q15, Q17, Q20, Q22, Q23, Q25, Q28, Q3, Q30, Q31: IRLIZ44N, TO220:TO-220-3_EXTENDED2, symbol Transistor_FET:IRLIZ44N
- removed R17, R19, R31, R32, R33, R35, R47, R48, R49, R51, R63, R64: 10k, TO220:R_Axial_Clean, symbol Device:R
- removed R18, R20, R21, R22, R23, R24, R25, R26, R27, R28, R29, R30, R34, R36, R37, R38, R39, R40, R41, R42, R43, R44, R45, R46, R50, R52, R53, R54, R55, R56, R57, R58, R59, R60, R61, R62: 1k, TO220:R_Axial_Clean, symbol Device:R
- removed U10, U11, U16, U17, U22, U23: LM5109MA, Package_SO:SOIC-8_3.9x4.9mm_P1.27mm, symbol Driver_FET:LM5109MA
- removed U12, U15, U18, U21, U24, U9: BTN7960B, termocuplu:IC_BTN7960B, symbol ktype:BTN7960B
- removed U13, U14, U19, U20, U25, U4: IR2110, Package_DIP:DIP-14_W7.62mm, symbol Driver_FET:IR2110
- AMS11173V3: footprint Package_TO_SOT_THT:TO-220-3_Horizontal_TabDown -> Footprints:TO-220-3_Horizontal_TabDown
- C1, C10, C11, C13, C14, C3, C5, C7, C9: footprint Capacitor_THT:C_Rect_L7.0mm_W3.5mm_P5.00mm -> Footprints:C_Rect_L7.0mm_W3.5mm_P5.00mm
- C12, C15, C2, C4, C6, C8: footprint termocuplu:CP_Elec_6.3x3.9_COMPOSITE -> Footprints:CP_Elec_6.3x3.9_COMPOSITE
- D1, D2, D3, D4, D5, D6: footprint Diode_THT:D_DO-41_SOD81_P10.16mm_Horizontal -> Footprints:D_DO-41_SOD81_P10.16mm_Horizontal
- H1, H2, H3, H4, H5, H6, H7, H8: footprint MountingHole:MountingHole_2.7mm_M2.5_Pad_Via -> Footprints:MountingHole_2.7mm_M2.5_Pad_Via
- J1, J2, J3, J5: footprint TO220:TerminalBlock_CLEAN_2PIN -> Footprints:TerminalBlock_CLEAN_2PIN
- Q1, Q5, Q6, Q8: footprint TO220:TO-220-3_EXTENDED2 -> Footprints:TO-220-3_EXTENDED2
- Q10, Q2, Q4, Q9: footprint Package_TO_SOT_SMD:TO-263-2 -> Footprints:TO-263-2
- R1, R10, R11, R12, R13, R14, R15, R16, R2, R3, R4, R5, R6, R7, R8, R9: footprint TO220:R_Axial_Clean -> Footprints:R_Axial_Clean
- TO_220Wiring1: footprint Connector_PinHeader_2.54mm:PinHeader_1x03_P2.54mm_Vertical -> Footprints:PinHeader_1x03_P2.54mm_Vertical
- U1, U6: footprint Package_DIP:DIP-14_W7.62mm -> Footprints:DIP-14_W7.62mm
- U2, U5: footprint Package_SO:SOIC-8_3.9x4.9mm_P1.27mm -> Footprints:SOIC-8_3.9x4.9mm_P1.27mm
- U3: footprint Package_TO_SOT_SMD:TO-252-2 -> Footprints:TO-252-2
- U7, U8: footprint termocuplu:IC_BTN7960B -> Footprints:IC_BTN7960B
Other:
- note removed: "Motor 2"
- note removed: "Motor 3"
- note removed: "Motor 4"
